File: luciannaFacundo.sch (KiCad schematic (older format))
At the start: 0 parts

Commit message: Correcciones
Parts:
- added FID101, FID102, FID103, FID104, FID105, FID106: Fiducial, Fiducial:Fiducial_1mm_Mask3mm, symbol Mechanical:Fiducial
- added LOGO101: Logo_Open_Hardware, Symbol:OSHW-Logo2_7.3x6mm_SilkScreen, symbol Graphic:Logo_Open_Hardware_Small
- added LOGO102: Logo_Kicad, Symbol:KiCad-Logo2_5mm_SilkScreen, symbol Graphic:Logo_Open_Hardware_Small
Other:
- note added: "Miscelaneos"
Changed lines of the file:
@@
 Title "Replica ESP32 Thing"
 Date "2019-06-04"
-Rev "Piza AG"
-Comp "Facundo A Lucianna"
+Rev "1.1"
+Comp "Autor: Facundo A Lucianna - Revisor: Alvaro Gabriel Pizá"
 Comment1 "https://creativecommons.org/licenses/by-sa/4.0/"
 Comment2 "Modificación sin el respaldo del autor original"
@@
 Wire Notes Line
 	3800 4350 3800 5550
+$Comp
+L Mechanical:Fiducial FID104
+U 1 1 5D11788B
+P 2100 6900
+F 0 "FID104" H 2185 6946 50  0000 L CNN
+F 1 "Fiducial" H 2185 6855 50  0000 L CNN
+F 2 "Fiducial:Fiducial_1mm_Mask3mm" H 2100 6900 50  0001 C CNN
+F 3 "~" H 2100 6900 50  0001 C CNN
+	1    2100 6900
+	1    0    0    -1
+$EndComp
+$Comp
+L Mechanical:Fiducial FID103
+U 1 1 5D1176F1
+P 2100 6600
+F 0 "FID103" H 2185 6646 50  0000 L CNN
+F 1 "Fiducial" H 2185 6555 50  0000 L CNN
+F 2 "Fiducial:Fiducial_1mm_Mask3mm" H 2100 6600 50  0001 C CNN
+F 3 "~" H 2100 6600 50  0001 C CNN
+	1    2100 6600
+	1    0    0    -1
+$EndComp
+$Comp
+L Mechanical:Fiducial FID101
+U 1 1 5D117419
+P 1400 6600
+F 0 "FID101" H 1485 6646 50  0000 L CNN
+F 1 "Fiducial" H 1485 6555 50  0000 L CNN
+F 2 "Fiducial:Fiducial_1mm_Mask3mm" H 1400 6600 50  0001 C CNN
+F 3 "~" H 1400 6600 50  0001 C CNN
+	1    1400 6600
+	1    0    0    -1
+$EndComp
+$Comp
+L Mechanical:Fiducial FID102
+U 1 1 5D116A37
+P 1400 6900
+F 0 "FID102" H 1485 6946 50  0000 L CNN
+F 1 "Fiducial" H 1485 6855 50  0000 L CNN
+F 2 "Fiducial:Fiducial_1mm_Mask3mm" H 1400 6900 50  0001 C CNN
+F 3 "~" H 1400 6900 50  0001 C CNN
+	1    1400 6900
+	1    0    0    -1
+$EndComp
+Text Notes 1350 6300 0    79   ~ 16
+Miscelaneos
+Wire Notes Line
+	1200 7150 1200 6100
+$Comp
+L Mechanical:Fiducial FID106
+U 1 1 5D117998
+P 2850 6900
+F 0 "FID106" H 2935 6946 50  0000 L CNN
+F 1 "Fiducial" H 2935 6855 50  0000 L CNN
+F 2 "Fiducial:Fiducial_1mm_Mask3mm" H 2850 6900 50  0001 C CNN
+F 3 "~" H 2850 6900 50  0001 C CNN
+	1    2850 6900
+	1    0    0    -1
+$EndComp
+$Comp
+L Mechanical:Fiducial FID105
+U 1 1 5D117A83
+P 2850 6600
+F 0 "FID105" H 2935 6646 50  0000 L CNN
+F 1 "Fiducial" H 2935 6555 50  0000 L CNN
+F 2 "Fiducial:Fiducial_1mm_Mask3mm" H 2850 6600 50  0001 C CNN
+F 3 "~" H 2850 6600 50  0001 C CNN
+	1    2850 6600
+	1    0    0    -1
+$EndComp
+$Comp
+L Graphic:Logo_Open_Hardware_Small LOGO101
+U 1 1 5D542AD4
+P 3950 6800
+F 0 "LOGO101" H 3950 7186 50  0000 C CNN
+F 1 "Logo_Open_Hardware" H 3950 7095 50  0000 C CNN
+F 2 "Symbol:OSHW-Logo2_7.3x6mm_SilkScreen" H 3950 6800 50  0001 C CNN
+F 3 "~" H 3950 6800 50  0001 C CNN
+	1    3950 6800
+	1    0    0    -1
+$EndComp
+$Comp
+L Graphic:Logo_Open_Hardware_Small LOGO102
+U 1 1 5D542EBF
+P 4900 6800
+F 0 "LOGO102" H 4750 7200 50  0000 L CNN
+F 1 "Logo_Kicad" H 4700 7100 50  0000 L CNN
+F 2 "Symbol:KiCad-Logo2_5mm_SilkScreen" H 4900 6800 50  0001 C CNN
+F 3 "~" H 4900 6800 50  0001 C CNN
+	1    4900 6800
+	1    0    0    -1
+$EndComp
+Wire Notes Line
+	5750 6100 5750 7150
+Wire Notes Line
+	1200 6100 5750 6100
+Wire Notes Line
+	1200 7150 5750 7150
 $EndSCHEMATC
